File: HW/LEDs.kicad_sch (KiCad schematic)
At the start: 26 parts, among them Q1 Q_NMOS_GSD

Commit message: continue routing
Connections:
- net DATA_LED: no longer D1.4 (DIN), Q1.3 (D), R4.2
- new net DATA_LED_OUT: D1.4 (DIN), Q1.3 (D), R4.2
Changed lines of the file:
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@@
     (stroke (width 0) (type default) (color 0 0 0 0))
   )
-  (global_label "DATA_LED" (shape input) (at 52.705 101.6 180) (fields_autoplaced)
+  (global_label "DATA_LED_OUT" (shape input) (at 52.705 101.6 180) (fields_autoplaced)
     (effects (font (size 1.27 1.27)) (justify right))
-    (property "Intersheet References" "${INTERSHEET_REFS}" (id 0) (at 41.4624 101.6794 0)
+    (property "Intersheet References" "${INTERSHEET_REFS}" (id 0) (at 36.8662 101.5206 0)
       (effects (font (size 1.27 1.27)) (justify right) hide)
     )
   )
-  (global_label "DATA_LED" (shape input) (at 75.565 71.12 0) (fields_autoplaced)
+  (global_label "DATA_LED_OUT" (shape input) (at 75.565 71.12 0) (fields_autoplaced)
     (effects (font (size 1.27 1.27)) (justify left))
-    (property "Intersheet References" "${INTERSHEET_REFS}" (id 0) (at 86.8076 71.0406 0)
+    (property "Intersheet References" "${INTERSHEET_REFS}" (id 0) (at 91.4038 71.0406 0)
       (effects (font (size 1.27 1.27)) (justify left) hide)
     )

Commit message: routed top PCB (with buttons, LEDs and phototransistor)
Changed lines of the file:
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@@
+    (stroke (width 0) (type default) (color 0 0 0 0))
+  )
+  (wire (pts (xy 57.785 85.725) (xy 57.785 83.82))
     (stroke (width 0) (type default) (color 0 0 0 0))
   )
   (wire (pts (xy 220.345 110.49) (xy 220.345 111.76))
+    (stroke (width 0) (type default) (color 0 0 0 0))
+  )
+  (wire (pts (xy 57.785 83.82) (xy 52.705 83.82))
     (stroke (width 0) (type default) (color 0 0 0 0))
   )
@@
     )
   )
+  (hierarchical_label "GND" (shape input) (at 52.705 83.82 180)
+    (effects (font (size 1.27 1.27)) (justify right))
+  )
   (hierarchical_label "DATA_LED" (shape input) (at 48.26 71.12 180)
     (effects (font (size 1.27 1.27)) (justify right))
@@
     (pin "4")
   )
+  (symbol (lib_id "power:GND") (at 57.785 85.725 0) (unit 1)
+    (in_bom yes) (on_board yes) (fields_autoplaced)
+    (property "Reference" "#PWR0198" (id 0) (at 57.785 92.075 0)
+      (effects (font (size 1.27 1.27)) hide)
+    )
+    (property "Value" "GND" (id 1) (at 57.785 90.1684 0))
+    (property "Footprint" "" (id 2) (at 57.785 85.725 0)
+      (effects (font (size 1.27 1.27)) hide)
+    )
+    (property "Datasheet" "" (id 3) (at 57.785 85.725 0)
+      (effects (font (size 1.27 1.27)) hide)
+    )
+    (pin "1")
+  )
   (symbol (lib_id "LED:WS2812B") (at 169.545 138.43 0) (unit 1)

Commit message: 2 PCB version of Semafor done
Changed lines of the file:
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@@
   (junction (at 170.815 92.71) (diameter 0) (color 0 0 0 0)
   )
+  (junction (at 57.785 83.82) (diameter 0) (color 0 0 0 0)
+  )
   (junction (at 69.215 71.12) (diameter 0) (color 0 0 0 0)
+  )
+  (junction (at 56.515 33.02) (diameter 0) (color 0 0 0 0)
   )
   (junction (at 55.245 46.99) (diameter 0) (color 0 0 0 0)
@@
     (stroke (width 0) (type default) (color 0 0 0 0))
   )
+  (wire (pts (xy 57.785 83.82) (xy 60.325 83.82))
+    (stroke (width 0) (type default) (color 0 0 0 0))
+  )
   (wire (pts (xy 254.635 129.54) (xy 236.855 129.54))
     (stroke (width 0) (type default) (color 0 0 0 0))
@@
     (stroke (width 0) (type default) (color 0 0 0 0))
   )
+  (wire (pts (xy 56.515 33.02) (xy 56.515 35.56))
+    (stroke (width 0) (type default) (color 0 0 0 0))
+  )
   (wire (pts (xy 169.545 128.27) (xy 169.545 129.54))
     (stroke (width 0) (type default) (color 0 0 0 0))
@@
     (stroke (width 0) (type default) (color 0 0 0 0))
   )
+  (wire (pts (xy 56.515 33.02) (xy 58.42 33.02))
+    (stroke (width 0) (type default) (color 0 0 0 0))
+  )
   (wire (pts (xy 67.945 128.27) (xy 67.945 129.54))
     (stroke (width 0) (type default) (color 0 0 0 0))
@@
     (stroke (width 0) (type default) (color 0 0 0 0))
   )
-  (wire (pts (xy 56.515 30.48) (xy 56.515 35.56))
+  (wire (pts (xy 56.515 30.48) (xy 56.515 33.02))
     (stroke (width 0) (type default) (color 0 0 0 0))
   )
@@
     (pin "1")
   )
+  (symbol (lib_id "power:PWR_FLAG") (at 58.42 33.02 270) (unit 1)
+    (in_bom yes) (on_board yes) (fields_autoplaced)
+    (property "Reference" "#FLG0107" (id 0) (at 60.325 33.02 0)
+      (effects (font (size 1.27 1.27)) hide)
+    )
+    (property "Value" "PWR_FLAG" (id 1) (at 61.595 33.4538 90)
+      (effects (font (size 1.27 1.27)) (justify left))
+    )
+    (property "Footprint" "" (id 2) (at 58.42 33.02 0)
+      (effects (font (size 1.27 1.27)) hide)
+    )
+    (property "Datasheet" "~" (id 3) (at 58.42 33.02 0)
+      (effects (font (size 1.27 1.27)) hide)
+    )
+    (pin "1")
+  )
   (symbol (lib_id "Device:C") (at 256.54 98.425 0) (unit 1)
     (in_bom yes) (on_board yes) (fields_autoplaced)
@@
       (effects (font (size 1.27 1.27)) hide)
     )
+    (pin "1")
+  )
+  (symbol (lib_id "power:PWR_FLAG") (at 60.325 83.82 270) (unit 1)
+    (in_bom yes) (on_board yes) (fields_autoplaced)
+    (property "Reference" "#FLG0106" (id 0) (at 62.23 83.82 0)
+      (effects (font (size 1.27 1.27)) hide)
+    )
+    (property "Value" "PWR_FLAG" (id 1) (at 63.5 84.2538 90)
+      (effects (font (size 1.27 1.27)) (justify left))
+    )
+    (property "Footprint" "" (id 2) (at 60.325 83.82 0)
+      (effects (font (size 1.27 1.27)) hide)
+    )
+    (property "Datasheet" "~" (id 3) (at 60.325 83.82 0)
+      (effects (font (size 1.27 1.27)) hide)
+    )
