File: HW/v0.0/Semafor.kicad_pcb (KiCad board)
At the start: 2 copper layers, 148.8 x 160.7 mm, 93 parts, among them J1 USB_C_Receptacle_USB2.0, J2 USB_plug, M1 Motor_DC, Q1 Q_NMOS_GSD, Q2 Q_NMOS_GSD, Q3 Q_NMOS_GSD, Q4 Q_NMOS_GSD, SW6 SW_SPDT, U1 ESP32-C3, U2 CN3058E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

Commit message: add 3D models of my gadgets
Parts:
- SW6: moved to B.Cu
- turned SW6 to 90 degrees
Changed lines of the file:
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@@
-    )
-  )
-  (footprint "Connector_PinSocket_2.54mm:PinSocket_1x03_P2.54mm_Vertical" (layer "F.Cu")
-    (at -143.675 -75.325 -90)
-    (descr "Through hole straight socket strip, 1x03, 2.54mm pitch, single row (from Kicad 4.0.7), script generated")
-    (tags "Through hole socket strip THT 1x03 2.54mm single row")
-    (property "Sheetfile" "Semafor.kicad_sch")
-    (property "Sheetname" "")
-    (attr through_hole)
-    (fp_text reference "SW6" (at 0 -2.77 90) (layer "F.SilkS")
-      (effects (font (size 1 1) (thickness 0.15)))
-    )
-    (fp_text value "SW_SPDT" (at 0 7.85 90) (layer "F.Fab")
-      (effects (font (size 1 1) (thickness 0.15)))
-    )
-    (fp_text user "${REFERENCE}" (at 0 2.54) (layer "F.Fab")
-      (effects (font (size 1 1) (thickness 0.15)))
-    )
-    (fp_line (start 0 -1.33) (end 1.33 -1.33) (layer "F.SilkS") (width 0.12))
-    (fp_line (start 1.33 -1.33) (end 1.33 0) (layer "F.SilkS") (width 0.12))
-    (fp_line (start -1.33 6.41) (end 1.33 6.41) (layer "F.SilkS") (width 0.12))
-    (fp_line (start 1.33 1.27) (end 1.33 6.41) (layer "F.SilkS") (width 0.12))
-    (fp_line (start -1.33 1.27) (end -1.33 6.41) (layer "F.SilkS") (width 0.12))
-    (fp_line (start -1.33 1.27) (end 1.33 1.27) (layer "F.SilkS") (width 0.12))
-    (fp_line (start 1.75 6.85) (end -1.8 6.85) (layer "F.CrtYd") (width 0.05))
-    (fp_line (start 1.75 -1.8) (end 1.75 6.85) (layer "F.CrtYd") (width 0.05))
-    (fp_line (start -1.8 6.85) (end -1.8 -1.8) (layer "F.CrtYd") (width 0.05))
-    (fp_line (start -1.8 -1.8) (end 1.75 -1.8) (layer "F.CrtYd") (width 0.05))
-    (fp_line (start -1.27 -1.27) (end 0.635 -1.27) (layer "F.Fab") (width 0.1))
-    (fp_line (start 1.27 6.35) (end -1.27 6.35) (layer "F.Fab") (width 0.1))
-    (fp_line (start 1.27 -0.635) (end 1.27 6.35) (layer "F.Fab") (width 0.1))
-    (fp_line (start -1.27 6.35) (end -1.27 -1.27) (layer "F.Fab") (width 0.1))
-    (fp_line (start 0.635 -1.27) (end 1.27 -0.635) (layer "F.Fab") (width 0.1))
-    (pad "1" thru_hole rect (at 0 0 270) (size 1.7 1.7) (drill 1) (layers *.Cu *.Mask)
-      (net 33 "unconnected-(SW6-Pad1)") (pinfunction "A") (pintype "passive+no_connect"))
-    (pad "2" thru_hole oval (at 0 2.54 270) (size 1.7 1.7) (drill 1) (layers *.Cu *.Mask)
-      (net 67 "Net-(BT1-Pad1)") (pinfunction "B") (pintype "passive"))
-    (pad "3" thru_hole oval (at 0 5.08 270) (size 1.7 1.7) (drill 1) (layers *.Cu *.Mask)
-      (net 19 "+3V3") (pinfunction "C") (pintype "passive"))
-    (model "${KICAD6_3DMODEL_DIR}/Connector_PinSocket_2.54mm.3dshapes/PinSocket_1x03_P2.54mm_Vertical.step"
-      (offset (xyz 0 0 0))
-      (scale (xyz 1 1 1))
-      (rotate (xyz 0 0 0))
     )
   )
@@
     (pad "10" thru_hole rect (at 7 -15 315) (size 1.5 2) (drill 0.9) (layers *.Cu *.Mask)
       (net 1 "GND") (pinfunction "GND") (pintype "input"))
+    (model "D:/School/FEKT/Magisterske/Diplomka/dily_DPS/E22_900T22D.STEP"
+      (offset (xyz 0 0 0))
+      (scale (xyz 1 1 1))
+      (rotate (xyz 0 0 -90))
+    )
   )
   (footprint "Diode_SMD:D_SOD-123" (layer "B.Cu")
@@
       (net 59 "Net-(D23-Pad2)") (pinfunction "A") (pintype "passive"))
     (model "${KICAD6_3DMODEL_DIR}/Diode_SMD.3dshapes/D_SOD-123.step"
+      (offset (xyz 0 0 0))
+      (scale (xyz 1 1 1))
+      (rotate (xyz 0 0 0))
+    )
+  )
+  (footprint "Connector_PinSocket_2.54mm:PinSocket_1x03_P2.54mm_Vertical" (layer "B.Cu")
+    (at -143.675 -75.375 90)
+    (descr "Through hole straight socket strip, 1x03, 2.54mm pitch, single row (from Kicad 4.0.7), script generated")
+    (tags "Through hole socket strip THT 1x03 2.54mm single row")
+    (property "Sheetfile" "Semafor.kicad_sch")
+    (property "Sheetname" "")
+    (attr through_hole)
+    (fp_text reference "SW6" (at 0 2.77 90) (layer "B.SilkS")
+      (effects (font (size 1 1) (thickness 0.15)) (justify mirror))
+    )
+    (fp_text value "SW_SPDT" (at 0 -7.85 90) (layer "B.Fab")
+      (effects (font (size 1 1) (thickness 0.15)) (justify mirror))
+    )
+    (fp_text user "${REFERENCE}" (at 0 -2.54) (layer "B.Fab")
+      (effects (font (size 1 1) (thickness 0.15)) (justify mirror))
+    )
+    (fp_line (start 0 1.33) (end 1.33 1.33) (layer "B.SilkS") (width 0.12))
+    (fp_line (start 1.33 1.33) (end 1.33 0) (layer "B.SilkS") (width 0.12))
+    (fp_line (start -1.33 -6.41) (end 1.33 -6.41) (layer "B.SilkS") (width 0.12))
+    (fp_line (start 1.33 -1.27) (end 1.33 -6.41) (layer "B.SilkS") (width 0.12))
+    (fp_line (start -1.33 -1.27) (end -1.33 -6.41) (layer "B.SilkS") (width 0.12))
+    (fp_line (start -1.33 -1.27) (end 1.33 -1.27) (layer "B.SilkS") (width 0.12))
+    (fp_line (start 1.75 -6.85) (end -1.8 -6.85) (layer "B.CrtYd") (width 0.05))
+    (fp_line (start 1.75 1.8) (end 1.75 -6.85) (layer "B.CrtYd") (width 0.05))
+    (fp_line (start -1.8 -6.85) (end -1.8 1.8) (layer "B.CrtYd") (width 0.05))
+    (fp_line (start -1.8 1.8) (end 1.75 1.8) (layer "B.CrtYd") (width 0.05))
+    (fp_line (start -1.27 1.27) (end 0.635 1.27) (layer "B.Fab") (width 0.1))
+    (fp_line (start 1.27 -6.35) (end -1.27 -6.35) (layer "B.Fab") (width 0.1))
+    (fp_line (start 1.27 0.635) (end 1.27 -6.35) (layer "B.Fab") (width 0.1))
+    (fp_line (start -1.27 -6.35) (end -1.27 1.27) (layer "B.Fab") (width 0.1))
+    (fp_line (start 0.635 1.27) (end 1.27 0.635) (layer "B.Fab") (width 0.1))
+    (pad "1" thru_hole rect (at 0 0 90) (size 1.7 1.7) (drill 1) (layers *.Cu *.Mask)
+      (net 33 "unconnected-(SW6-Pad1)") (pinfunction "A") (pintype "passive+no_connect"))
+    (pad "2" thru_hole oval (at 0 -2.54 90) (size 1.7 1.7) (drill 1) (layers *.Cu *.Mask)
+      (net 67 "Net-(BT1-Pad1)") (pinfunction "B") (pintype "passive"))
+    (pad "3" thru_hole oval (at 0 -5.08 90) (size 1.7 1.7) (drill 1) (layers *.Cu *.Mask)
+      (net 19 "+3V3") (pinfunction "C") (pintype "passive"))
+    (model "${KICAD6_3DMODEL_DIR}/Connector_PinSocket_2.54mm.3dshapes/PinSocket_1x03_P2.54mm_Vertical.step"
       (offset (xyz 0 0 0))
       (scale (xyz 1 1 1))
@@
       (rotate (xyz 0 0 0))
     )
+    (model "D:/School/FEKT/Magisterske/Diplomka/dily_DPS/USB_C.STEP"
+      (offset (xyz 0 0 0))
+      (scale (xyz 1 1 1))
+      (rotate (xyz 0 0 90))
+    )
   )
   (footprint "Library:battery_dock" (layer "B.Cu")
@@
     (pad "2" thru_hole oval (at -36.35 -0.05 180) (size 1.524 2.9) (drill oval 0.762 1.6) (layers *.Cu *.Mask)
       (net 1 "GND") (pinfunction "-") (pintype "passive"))
+    (model "D:/School/FEKT/Magisterske/Diplomka/dily_DPS/Battery_pack.STEP"
+      (offset (xyz 0 0 0))
+      (scale (xyz 1 1 1))
+      (rotate (xyz 0 0 0))
+    )
   )
   (footprint "LED_SMD:LED_0603_1608Metric" (layer "B.Cu")
